File: kicad/AlexJ_bz_ArduinoGigaShield.kicad_pcb (KiCad board)
At the start: 2 copper layers, 155 x 90 mm, 59 parts, among them J1 Conn_01x08, J10 JSIDE_5V, J2 Conn_01x10, J3 Conn_01x08, J4 Conn_01x08, J5 Conn_01x26, J6 Conn_01x08, J7 Conn_01x08, J8 Conn_01x26, J9 JSIDE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

Commit message: Update KiCad schematic and PCB annotations for v0.2 IC replacements
Schematic: Update Value, Datasheet, and Description properties on U1-U5
to reflect new IC types (SN74LVC541, SN74AHCT541, SN74LVC4245A).
Update U5 Footprint property to TSSOP-24.

PCB: Update Value, Datasheet, and Description on U1-U5 footprints.
Update U5 footprint reference to TSSOP-24. Change silkscreen from
V0.1 to V0.2.

Note: lib_symbol definitions, pin mappings, footprint geometry, and
trace routing still reference TXB0108PW and must be updated in
KiCad GUI. See CHANGES-V0.2.md for full implementation guide.
Parts:
- U1, U2, U3: value TXB0108PW -> SN74LVC541
- U4: value TXB0108PW -> SN74AHCT541
- U5: value TXB0108PW -> SN74LVC4245A; footprint Package_SO:TSSOP-20_4.4x6.5mm_P0.65mm -> Package_SO:TSSOP-24_4.4x7.8mm_P0.65mm
Other:
- board text added: "ARDUINO GIGA R1 SHIELD V0.2"
- board text removed: "ARDUINO GIGA R1 SHIELD V0.1"
Changed lines of the file:
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@@
 			)
 		)
-		(property "Value" "TXB0108PW"
+		(property "Value" "SN74LVC541"
 			(at 0 4.2 90)
 			(layer "F.Fab")
@@
 			)
 		)
-		(property "Datasheet" "http://www.ti.com/lit/ds/symlink/txb0108.pdf"
+		(property "Datasheet" "https://www.ti.com/lit/ds/symlink/sn74lvc541a.pdf"
 			(at 0 0 90)
 			(layer "F.Fab")
@@
 			)
 		)
-		(property "Description" "8-Bit Bidirectional Voltage-Level Translator, Auto Direction Sensing and ±15-kV ESD Protection, 1.2 - 3.6V APort, 1.65 - 5.5V BPort, TSSOP-20"
+		(property "Description" "Octal Buffer/Driver With 3-State Outputs, 5V-Tolerant Inputs, TSSOP-20 (v0.2: control inputs MREQ/IORQ/RD/WR)"
 			(at 0 0 90)
 			(layer "F.Fab")
@@
 			)
 		)
-		(property "Value" "TXB0108PW"
+		(property "Value" "SN74LVC541"
 			(at 0 4.2 0)
 			(layer "F.Fab")
@@
 			)
 		)
-		(property "Datasheet" "http://www.ti.com/lit/ds/symlink/txb0108.pdf"
+		(property "Datasheet" "https://www.ti.com/lit/ds/symlink/sn74lvc541a.pdf"
 			(at 0 0 0)
 			(layer "F.Fab")
@@
 			)
 		)
-		(property "Description" "8-Bit Bidirectional Voltage-Level Translator, Auto Direction Sensing and ±15-kV ESD Protection, 1.2 - 3.6V APort, 1.65 - 5.5V BPort, TSSOP-20"
+		(property "Description" "Octal Buffer/Driver With 3-State Outputs, 5V-Tolerant Inputs, TSSOP-20 (v0.2: address bus A8-A15)"
 			(at 0 0 0)
 			(layer "F.Fab")
@@
 		)
 	)
-	(footprint "Package_SO:TSSOP-20_4.4x6.5mm_P0.65mm"
+	(footprint "Package_SO:TSSOP-24_4.4x7.8mm_P0.65mm"
 		(layer "F.Cu")
 		(at 195.78 45.69 90)
-		(descr "TSSOP, 20 Pin (JEDEC MO-153 Var AC https://www.jedec.org/document_search?search_api_views_fulltext=MO-153), generated with kicad-footprint-generator ipc_gullwing_generator.py")
+		(descr "TSSOP, 24 Pin (4.4x7.8mm, 0.65mm pitch), v0.2 replacement for TXB0108PW - SN74LVC4245A bidirectional bus transceiver with DIR pin")
 		(tags "TSSOP SO")
 		(property "Reference" "U5"
@@
 			)
 		)
-		(property "Value" "TXB0108PW"
+		(property "Value" "SN74LVC4245A"
 			(at 0 4.2 90)
 			(layer "F.Fab")
@@
 			)
 		)
-		(property "Datasheet" "http://www.ti.com/lit/ds/symlink/txb0108.pdf"
+		(property "Datasheet" "https://www.ti.com/lit/ds/symlink/sn74lvc4245a.pdf"
 			(at 0 0 90)
 			(layer "F.Fab")
@@
 			)
 		)
-		(property "Description" "8-Bit Bidirectional Voltage-Level Translator, Auto Direction Sensing and ±15-kV ESD Protection, 1.2 - 3.6V APort, 1.65 - 5.5V BPort, TSSOP-20"
+		(property "Description" "8-Bit Dual-Supply Bus Transceiver With Configurable Voltage Translation and 3-State Outputs, TSSOP-24 (v0.2: data bus D0-D7, DIR on Arduino D2)"
 			(at 0 0 90)
 			(layer "F.Fab")
@@
 			)
 		)
-		(property ki_fp_filters "TSSOP*4.4x6.5mm*P0.65mm*")
+		(property ki_fp_filters "TSSOP*4.4x7.8mm*P0.65mm*")
 		(sheetname "/")
 		(sheetfile "AlexJ_bz_ArduinoGigaShield.kicad_sch")
@@
 			)
 		)
-		(property "Value" "TXB0108PW"
+		(property "Value" "SN74AHCT541"
 			(at 0 4.2 0)
 			(layer "F.Fab")
@@
 			)
 		)
-		(property "Datasheet" "http://www.ti.com/lit/ds/symlink/txb0108.pdf"
+		(property "Datasheet" "https://www.ti.com/lit/ds/symlink/sn74ahct541.pdf"
 			(at 0 0 0)
 			(layer "F.Fab")
@@
 			)
 		)
-		(property "Description" "8-Bit Bidirectional Voltage-Level Translator, Auto Direction Sensing and ±15-kV ESD Protection, 1.2 - 3.6V APort, 1.65 - 5.5V BPort, TSSOP-20"
+		(property "Description" "Octal Buffer/Driver With 3-State Outputs, TTL-Compatible Inputs, TSSOP-20 (v0.2: control outputs CLK/RESET/INT/NMI)"
 			(at 0 0 0)
 			(layer "F.Fab")
@@
 			)
 		)
-		(property "Value" "TXB0108PW"
+		(property "Value" "SN74LVC541"
 			(at 0 4.2 90)
 			(layer "F.Fab")
@@
 			)
 		)
-		(property "Datasheet" "http://www.ti.com/lit/ds/symlink/txb0108.pdf"
+		(property "Datasheet" "https://www.ti.com/lit/ds/symlink/sn74lvc541a.pdf"
 			(at 0 0 90)
 			(layer "F.Fab")
@@
 			)
 		)
-		(property "Description" "8-Bit Bidirectional Voltage-Level Translator, Auto Direction Sensing and ±15-kV ESD Protection, 1.2 - 3.6V APort, 1.65 - 5.5V BPort, TSSOP-20"
+		(property "Description" "Octal Buffer/Driver With 3-State Outputs, 5V-Tolerant Inputs, TSSOP-20 (v0.2: address bus A0-A7)"
 			(at 0 0 90)
 			(layer "F.Fab")
@@
 		)
 	)
-	(gr_text "ARDUINO GIGA R1 SHIELD V0.1"
+	(gr_text "ARDUINO GIGA R1 SHIELD V0.2"
 		(at 111.77 94.26 90)
 		(layer "F.SilkS")
